File: ac-shifter.kicad_sch (KiCad schematic)
At the start: 12 parts, among them U13 LM393

Commit message: schem: add part numbers to BOM
Parts:
- C45: Basic (none) -> Y; JLCPCB Part # (none) -> C15849; Manufacturer (none) -> Samsung Electro-Mechanics; Manufacturer Part Number (none) -> CL10A105KB8NNNC
- C46: Basic (none) -> Y; JLCPCB Part # (none) -> C307331; Manufacturer (none) -> Samsung Electro-Mechanics; Manufacturer Part Number (none) -> CL05B104KB54PNC
- C47: Basic (none) -> Y; JLCPCB Part # (none) -> C52923; Manufacturer (none) -> Samsung Electro-Mechanics; Manufacturer Part Number (none) -> CL05A105KA5NQNC
- D8: Basic (none) -> Y; JLCPCB Part # (none) -> C2488; Manufacturer (none) -> Microdiode Semiconductor (MDD); Manufacturer Part Number (none) -> C2488
- TP1, TP4, TP7: now left out of the parts list
Changed lines of the file:
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@@
+			)
+		)
+		(property "Basic" "Y"
+			(at 115.57 57.15 0)
+			(effects
+				(font
+					(size 1.27 1.27)
+				)
+				(hide yes)
+			)
+		)
+		(property "JLCPCB Part #" "C307331"
+			(at 115.57 57.15 0)
+			(effects
+				(font
+					(size 1.27 1.27)
+				)
+				(hide yes)
+			)
+		)
+		(property "Manufacturer" "Samsung Electro-Mechanics "
+			(at 115.57 57.15 0)
+			(effects
+				(font
+					(size 1.27 1.27)
+				)
+				(hide yes)
+			)
+		)
+		(property "Manufacturer Part Number" "CL05B104KB54PNC"
+			(at 115.57 57.15 0)
+			(effects
+				(font
+					(size 1.27 1.27)
+				)
+				(hide yes)
 			)
 		)
@@
 			)
 		)
+		(property "Basic" "Y"
+			(at 92.71 93.98 0)
+			(effects
+				(font
+					(size 1.27 1.27)
+				)
+				(hide yes)
+			)
+		)
+		(property "JLCPCB Part #" "C2488"
+			(at 92.71 93.98 0)
+			(effects
+				(font
+					(size 1.27 1.27)
+				)
+				(hide yes)
+			)
+		)
+		(property "Manufacturer" "Microdiode Semiconductor (MDD)"
+			(at 92.71 93.98 0)
+			(effects
+				(font
+					(size 1.27 1.27)
+				)
+				(hide yes)
+			)
+		)
+		(property "Manufacturer Part Number" "C2488"
+			(at 92.71 93.98 0)
+			(effects
+				(font
+					(size 1.27 1.27)
+				)
+				(hide yes)
+			)
+		)
 		(pin "3"
 		)
@@
 		(unit 1)
 		(exclude_from_sim no)
-		(in_bom yes)
+		(in_bom no)
 		(on_board yes)
 		(dnp no)
@@
 			)
 		)
+		(property "Basic" "Y"
+			(at 129.54 100.33 0)
+			(effects
+				(font
+					(size 1.27 1.27)
+				)
+				(hide yes)
+			)
+		)
+		(property "JLCPCB Part #" "C52923"
+			(at 129.54 100.33 0)
+			(effects
+				(font
+					(size 1.27 1.27)
+				)
+				(hide yes)
+			)
+		)
+		(property "Manufacturer" "Samsung Electro-Mechanics "
+			(at 129.54 100.33 0)
+			(effects
+				(font
+					(size 1.27 1.27)
+				)
+				(hide yes)
+			)
+		)
+		(property "Manufacturer Part Number" "CL05A105KA5NQNC"
+			(at 129.54 100.33 0)
+			(effects
+				(font
+					(size 1.27 1.27)
+				)
+				(hide yes)
+			)
+		)
 		(pin "1"
 		)
@@
 			)
 		)
+		(property "Basic" "Y"
+			(at 109.22 100.33 0)
+			(effects
+				(font
+					(size 1.27 1.27)
+				)
+				(hide yes)
+			)
+		)
+		(property "JLCPCB Part #" "C15849"
+			(at 109.22 100.33 0)
+			(effects
+				(font
+					(size 1.27 1.27)
+				)
+				(hide yes)
+			)
+		)
+		(property "Manufacturer" "Samsung Electro-Mechanics "
+			(at 109.22 100.33 0)
+			(effects
+				(font
+					(size 1.27 1.27)
+				)
+				(hide yes)
+			)
+		)
+		(property "Manufacturer Part Number" "CL10A105KB8NNNC"
+			(at 109.22 100.33 0)
+			(effects
+				(font
+					(size 1.27 1.27)
+				)
+				(hide yes)
+			)
+		)
 		(pin "1"
 		)
@@
 		(unit 1)
 		(exclude_from_sim no)
-		(in_bom yes)
+		(in_bom no)
 		(on_board yes)
 		(dnp no)
@@
 		(unit 1)
 		(exclude_from_sim no)
-		(in_bom yes)
-		(on_board yes)
-		(dnp no)
+		(in_bom no)
+		(on_board yes)
+		(dnp no)

Commit message: schem: add remaining part numbers to BOM
Parts:
- R53: Basic (none) -> Y; JLCPCB Part # (none) -> C22809; Manufacturer (none) -> Uniroyal Elec; Manufacturer Part Number (none) -> 0603WAF1502T5E
- R54, R55, R56: Basic (none) -> Y; JLCPCB Part # (none) -> C25804; Manufacturer (none) -> Uniroyal Elec; Manufacturer Part Number (none) -> 0603WAF1002T5E
- U13: Basic (none) -> Y; JLCPCB Part # (none) -> C7955; Manufacturer (none) -> onsemi; Manufacturer Part Number (none) -> LM393DR2G
